File: PCB/max31865_00.sch (KiCad schematic (older format))
At the start: 16 parts, among them J2 Conn_01x04, U6 MAX31865

Commit message: Patrick: 40-pin header -> 2x 24-pin header, holes added.
Parts:
- removed J2: Conn_01x04, TerminalBlock_4Ucon:TerminalBlock_4Ucon_1x04_P3.50mm_Horizontal, symbol Connector_Generic:Conn_01x04
- removed SJ1: SOLDERJUMPER_2WAY, Adafruit MAX31865:SOLDERJUMPER_2WAY_OPEN_NOPASTE, symbol Adafruit_MAX31865-eagle-import:SOLDERJUMPER_2WAY
- removed SJ2, SJ3: SOLDERJUMPER, Adafruit MAX31865:SOLDERJUMPER_ARROW_NOPASTE, symbol Adafruit_MAX31865-eagle-import:SOLDERJUMPER
Connections:
- net labels added: O1, O3, O5, O7
- wire segments 83 -> 57
- no-connect marks 0 -> 1
Other:
- note removed: "C3 = 100nF for 100 ohm RTD, 10nF for 1K"
- note removed: "SJ1 to GND for 2/4-wire, to FORCE+ for 3-wire"
- note removed: "SJ2 closed on 2/3-wire setups, open for 4-wire"
- moved on the sheet: C5, R4
Changed lines of the file:
@@
-GND
-Wire Wire Line
-	6500 3600 6700 3600
-Wire Wire Line
-	6700 3600 6700 3400
-Wire Wire Line
-	6700 3400 6800 3400
-Text Label 6500 3600 0    10   ~ 0
 GND
 Wire Wire Line
@@
 	6200 2500 6400 2500
 Wire Wire Line
-	6400 2500 7000 2500
+	6400 2500 6900 2500
 Wire Wire Line
 	6200 2700 6400 2700
@@
 Connection ~ 6400 2500
 Wire Wire Line
-	6200 2900 7000 2900
-Wire Wire Line
-	6200 3100 7000 3100
-Wire Wire Line
-	7000 3100 7000 2900
-Connection ~ 7000 2900
-Wire Wire Line
-	6200 3700 6800 3700
-Wire Wire Line
-	6800 3800 6800 3700
-Wire Wire Line
-	7400 3700 7600 3700
-Wire Wire Line
-	7600 3700 7600 3400
-Wire Wire Line
-	6800 3700 7400 3700
-Connection ~ 6800 3700
-Connection ~ 7400 3700
-Wire Wire Line
-	6200 3300 6500 3300
-Wire Wire Line
-	6500 3400 6500 3300
-Wire Wire Line
-	6500 3300 7400 3300
-Connection ~ 6500 3300
-Connection ~ 7400 3300
-Wire Wire Line
-	6400 3500 6200 3500
-Wire Wire Line
-	7400 4500 7600 4500
-Wire Wire Line
-	7600 4500 7600 4200
-Wire Wire Line
-	6200 4400 6300 4400
-Wire Wire Line
-	6300 4400 6300 4500
-Wire Wire Line
-	6300 4500 7400 4500
-Connection ~ 7400 4500
-Wire Wire Line
-	7400 4100 7700 4100
-Wire Wire Line
-	6900 4200 6900 4100
-Wire Wire Line
-	6900 4200 6800 4200
-Wire Wire Line
-	6800 4200 6700 4200
-Wire Wire Line
-	6700 4200 6700 4100
-Wire Wire Line
-	6200 4200 6300 4200
-Wire Wire Line
-	6300 4200 6300 4100
-Wire Wire Line
-	6700 4100 6300 4100
-Wire Wire Line
-	6800 4100 6800 4200
-Wire Wire Line
-	7400 4100 6900 4100
-Connection ~ 7400 4100
-Connection ~ 6800 4200
+	6200 2900 6900 2900
+Wire Wire Line
+	6200 3100 6900 3100
+Wire Wire Line
+	6900 3100 6900 2900
+Connection ~ 6900 2900
+Wire Wire Line
+	6400 3800 6400 3700
+Wire Wire Line
+	6400 4100 6400 4200
 Wire Wire Line
 	4900 3000 4100 3000
@@
 L Adafruit_MAX31865-eagle-import:RESISTOR0805_NOOUTLINE R4
 U 1 1 5BC8807C
-P 7000 2700
-F 0 "R4" H 7000 2800 50  0000 C CNN
-F 1 "430Ω / 4300Ω 0.1%" H 7000 2600 40  0000 C CNB
-F 2 "Adafruit MAX31865:0805-NO" H 7000 2700 50  0001 C CNN
-F 3 "" H 7000 2700 50  0001 C CNN
-	1    7000 2700
+P 6900 2700
+F 0 "R4" H 6900 2800 50  0000 C CNN
+F 1 "430Ω / 4300Ω 0.1%" H 6900 2600 40  0000 C CNB
+F 2 "Adafruit MAX31865:0805-NO" H 6900 2700 50  0001 C CNN
+F 3 "" H 6900 2700 50  0001 C CNN
+	1    6900 2700
 	0    -1   -1   0
 $EndComp
@@
 L Adafruit_MAX31865-eagle-import:CAP_CERAMIC0805-NOOUTLINE C5
 U 1 1 5BC893CC
-P 6800 4000
-F 0 "C5" V 6710 4049 50  0000 C CNN
-F 1 "100nF" V 6890 4049 50  0000 C CNN
-F 2 "Adafruit MAX31865:0805-NO" H 6800 4000 50  0001 C CNN
-F 3 "" H 6800 4000 50  0001 C CNN
-	1    6800 4000
-	1    0    0    -1
-$EndComp
-$Comp
-L Adafruit_MAX31865-eagle-import:SOLDERJUMPER_2WAY SJ1
-U 1 1 5BC88097
-P 6500 3500
-F 0 "SJ1" H 6300 3350 59  0000 L BNN
-F 1 "SOLDERJUMPER_2WAY" H 6300 3250 59  0000 L BNN
-F 2 "Adafruit MAX31865:SOLDERJUMPER_2WAY_OPEN_NOPASTE" H 6500 3500 50  0001 C CNN
-F 3 "" H 6500 3500 50  0001 C CNN
-	1    6500 3500
-	0    -1   -1   0
-$EndComp
-$Comp
-L Adafruit_MAX31865-eagle-import:GND #U$010
-U 1 1 5BC880D9
-P 6800 3500
-F 0 "#U$010" H 6800 3500 50  0001 C CNN
-F 1 "GND" H 6740 3400 42  0000 L BNN
-F 2 "" H 6800 3500 50  0001 C CNN
-F 3 "" H 6800 3500 50  0001 C CNN
-	1    6800 3500
-	1    0    0    -1
-$EndComp
-$Comp
-L Adafruit_MAX31865-eagle-import:SOLDERJUMPER SJ2
-U 1 1 5BC880AE
-P 7400 3500
-F 0 "SJ2" H 7300 3600 59  0000 L BNN
-F 1 "SOLDERJUMPER" H 7300 3350 59  0000 L BNN
-F 2 "Adafruit MAX31865:SOLDERJUMPER_ARROW_NOPASTE" H 7400 3500 50  0001 C CNN
-F 3 "" H 7400 3500 50  0001 C CNN
-	1    7400 3500
-	0    -1   -1   0
-$EndComp
-$Comp
-L Adafruit_MAX31865-eagle-import:SOLDERJUMPER SJ3
-U 1 1 5BC880C1
-P 7400 4300
-F 0 "SJ3" H 7300 4400 59  0000 L BNN
-F 1 "SOLDERJUMPER" H 7300 4150 59  0000 L BNN
-F 2 "Adafruit MAX31865:SOLDERJUMPER_ARROW_NOPASTE" H 7400 4300 50  0001 C CNN
-F 3 "" H 7400 4300 50  0001 C CNN
-	1    7400 4300
-	0    -1   -1   0
+P 6400 4000
+F 0 "C5" V 6310 4049 50  0000 C CNN
+F 1 "100nF" V 6490 4049 50  0000 C CNN
+F 2 "Adafruit MAX31865:0805-NO" H 6400 4000 50  0001 C CNN
+F 3 "" H 6400 4000 50  0001 C CNN
+	1    6400 4000
+	1    0    0    -1
 $EndComp
 $Comp
@@
 	0    -1   -1   0
 $EndComp
-Text Notes 8400 3900 0    59   ~ 0
-C3 = 100nF for 100 ohm RTD, 10nF for 1K
-Text Notes 7200 2800 0    59   ~ 0
+Text Notes 7100 2800 0    59   ~ 0
 R1 = 4x RTD resistance at 0°C (so 400 ohm for a 100 ohm RTD).\nUse high quality 1% or better resistors
-Text Notes 6300 4800 0    59   ~ 0
-SJ1 to GND for 2/4-wire, to FORCE+ for 3-wire
-Text Notes 6300 5000 0    59   ~ 0
-SJ2 closed on 2/3-wire setups, open for 4-wire
 Text GLabel 2400 2400 0    50   Input ~ 0
 SDI_5V
@@
 Wire Wire Line
 	4900 2700 4750 2700
-$Comp
-L Connector_Generic:Conn_01x04 J2
-U 1 1 5BCA61C0
-P 8100 3400
-F 0 "J2" H 8180 3392 50  0000 L CNN
-F 1 "Conn_01x04" H 8180 3301 50  0000 L CNN
-F 2 "TerminalBlock_4Ucon:TerminalBlock_4Ucon_1x04_P3.50mm_Horizontal" H 8100 3400 50  0001 C CNN
-F 3 "~" H 8100 3400 50  0001 C CNN
-	1    8100 3400
-	1    0    0    -1
-$EndComp
-Wire Wire Line
-	7700 4100 7700 3500
-Wire Wire Line
-	7600 4200 7800 4200
-Wire Wire Line
-	7800 4200 7800 3600
-Wire Wire Line
-	7800 3600 7900 3600
-Wire Wire Line
-	7700 3500 7900 3500
-Wire Wire Line
-	7600 3400 7900 3400
-Wire Wire Line
-	7400 3300 7900 3300
+Wire Wire Line
+	6200 3300 6950 3300
+Wire Wire Line
+	6200 4400 6950 4400
+Wire Wire Line
+	6200 3700 6400 3700
+Wire Wire Line
+	6200 4200 6400 4200
+Text GLabel 6950 3300 2    50   Input ~ 0
+O1
+Text GLabel 6950 3700 2    50   Input ~ 0
+O3
+Text GLabel 6950 4200 2    50   Input ~ 0
+O5
+Text GLabel 6950 4400 2    50   Input ~ 0
+O7
+NoConn ~ 6200 3500
+Connection ~ 6400 3700
+Wire Wire Line
+	6400 3700 6950 3700
+Connection ~ 6400 4200
+Wire Wire Line
+	6400 4200 6950 4200
 $EndSCHEMATC
