File: PCB/max31865_04.sch (KiCad schematic (older format))
At the start: 16 parts, among them J6 Conn_01x04, U10 MAX31865

Commit message: Patrick: 40-pin header -> 2x 24-pin header, holes added.
Parts:
- removed J6: Conn_01x04, TerminalBlock_4Ucon:TerminalBlock_4Ucon_1x04_P3.50mm_Horizontal, symbol Connector_Generic:Conn_01x04
- removed SJ13: SOLDERJUMPER_2WAY, Adafruit MAX31865:SOLDERJUMPER_2WAY_OPEN_NOPASTE, symbol Adafruit_MAX31865-eagle-import:SOLDERJUMPER_2WAY
- removed SJ14, SJ15: SOLDERJUMPER, Adafruit MAX31865:SOLDERJUMPER_ARROW_NOPASTE, symbol Adafruit_MAX31865-eagle-import:SOLDERJUMPER
Connections:
- net labels added: O33, O35, O37, O39
- wire segments 83 -> 57
- no-connect marks 0 -> 1
Other:
- note removed: "SJ1 to GND for 2/4-wire, to FORCE+ for 3-wire"
- note removed: "SJ2 closed on 2/3-wire setups, open for 4-wire"
Changed lines of the file:
@@
-GND
-Wire Wire Line
-	6500 3600 6700 3600
-Wire Wire Line
-	6700 3600 6700 3400
-Wire Wire Line
-	6700 3400 6800 3400
-Text Label 6500 3600 0    10   ~ 0
 GND
 Wire Wire Line
@@
 Text Label 5600 1200 0    10   ~ 0
 VDD
-Wire Wire Line
-	6200 2500 6400 2500
-Wire Wire Line
-	6400 2500 7000 2500
-Wire Wire Line
-	6200 2700 6400 2700
-Wire Wire Line
-	6400 2700 6400 2500
-Connection ~ 6400 2500
-Wire Wire Line
-	6200 2900 7000 2900
-Wire Wire Line
-	6200 3100 7000 3100
-Wire Wire Line
-	7000 3100 7000 2900
-Connection ~ 7000 2900
-Wire Wire Line
-	6200 3700 6800 3700
-Wire Wire Line
-	6800 3800 6800 3700
-Wire Wire Line
-	6200 3300 6500 3300
-Wire Wire Line
-	6500 3400 6500 3300
-Wire Wire Line
-	6400 3500 6200 3500
-Wire Wire Line
-	6200 4400 6300 4400
-Wire Wire Line
-	6300 4400 6300 4500
-Wire Wire Line
-	6900 4200 6900 4100
-Wire Wire Line
-	6900 4200 6800 4200
-Wire Wire Line
-	6800 4200 6700 4200
-Wire Wire Line
-	6700 4200 6700 4100
-Wire Wire Line
-	6200 4200 6300 4200
-Wire Wire Line
-	6300 4200 6300 4100
-Wire Wire Line
-	6700 4100 6300 4100
-Wire Wire Line
-	6800 4100 6800 4200
-Connection ~ 6800 4200
 Wire Wire Line
 	4900 3000 4100 3000
@@
 F 3 "" H 5600 1100 50  0001 C CNN
 	1    5600 1100
-	1    0    0    -1
-$EndComp
-$Comp
-L Adafruit_MAX31865-eagle-import:RESISTOR0805_NOOUTLINE R20
-U 1 1 5BC8807D
-P 7000 2700
-F 0 "R20" H 7000 2800 50  0000 C CNN
-F 1 "430Ω / 4300Ω 0.1%" H 7000 2600 40  0000 C CNB
-F 2 "Adafruit MAX31865:0805-NO" H 7000 2700 50  0001 C CNN
-F 3 "" H 7000 2700 50  0001 C CNN
-	1    7000 2700
-	0    -1   -1   0
-$EndComp
-$Comp
-L Adafruit_MAX31865-eagle-import:CAP_CERAMIC0805-NOOUTLINE C17
-U 1 1 5BC880CA
-P 6800 4000
-F 0 "C17" V 6710 4049 50  0000 C CNN
-F 1 "100nF" V 6890 4049 50  0000 C CNN
-F 2 "Adafruit MAX31865:0805-NO" H 6800 4000 50  0001 C CNN
-F 3 "" H 6800 4000 50  0001 C CNN
-	1    6800 4000
-	1    0    0    -1
-$EndComp
-$Comp
-L Adafruit_MAX31865-eagle-import:SOLDERJUMPER_2WAY SJ13
-U 1 1 5BC8809A
-P 6500 3500
-F 0 "SJ13" H 6300 3350 59  0000 L BNN
-F 1 "SOLDERJUMPER_2WAY" H 6300 3250 59  0000 L BNN
-F 2 "Adafruit MAX31865:SOLDERJUMPER_2WAY_OPEN_NOPASTE" H 6500 3500 50  0001 C CNN
-F 3 "" H 6500 3500 50  0001 C CNN
-	1    6500 3500
-	0    -1   -1   0
-$EndComp
-$Comp
-L Adafruit_MAX31865-eagle-import:GND #U$038
-U 1 1 5BC880D5
-P 6800 3500
-F 0 "#U$038" H 6800 3500 50  0001 C CNN
-F 1 "GND" H 6740 3400 42  0000 L BNN
-F 2 "" H 6800 3500 50  0001 C CNN
-F 3 "" H 6800 3500 50  0001 C CNN
-	1    6800 3500
 	1    0    0    -1
 $EndComp
@@
 	0    -1   -1   0
 $EndComp
-Text Notes 7200 2800 0    59   ~ 0
-R1 = 4x RTD resistance at 0°C (so 400 ohm for a 100 ohm RTD).\nUse high quality 1% or better resistors
-Text Notes 6300 4800 0    59   ~ 0
-SJ1 to GND for 2/4-wire, to FORCE+ for 3-wire
-Text Notes 6300 5000 0    59   ~ 0
-SJ2 closed on 2/3-wire setups, open for 4-wire
 Text GLabel 2400 2400 0    50   Input ~ 0
 SDI_5V
@@
 	4900 2700 4750 2700
 Wire Wire Line
-	7400 3700 7600 3700
-Wire Wire Line
-	7600 3700 7600 3400
-Wire Wire Line
-	6800 3700 7400 3700
-Connection ~ 7400 3700
-Wire Wire Line
-	6500 3300 7400 3300
-Connection ~ 7400 3300
-Wire Wire Line
-	7400 4500 7600 4500
-Wire Wire Line
-	7600 4500 7600 4200
-Wire Wire Line
-	6300 4500 7400 4500
-Connection ~ 7400 4500
-Wire Wire Line
-	7400 4100 7700 4100
-Wire Wire Line
-	7400 4100 6900 4100
-Connection ~ 7400 4100
-$Comp
-L Adafruit_MAX31865-eagle-import:SOLDERJUMPER SJ?
-U 1 1 5BCCAE59
-P 7400 3500
-AR Path="/5BC99DB9/5BCCAE59" Ref="SJ?"  Part="1"
-AR Path="/5BCA1914/5BCCAE59" Ref="SJ14"  Part="1"
-F 0 "SJ14" H 7300 3600 59  0000 L BNN
-F 1 "SOLDERJUMPER" H 7300 3350 59  0000 L BNN
-F 2 "Adafruit MAX31865:SOLDERJUMPER_ARROW_NOPASTE" H 7400 3500 50  0001 C CNN
-F 3 "" H 7400 3500 50  0001 C CNN
-	1    7400 3500
-	0    -1   -1   0
-$EndComp
-$Comp
-L Adafruit_MAX31865-eagle-import:SOLDERJUMPER SJ?
-U 1 1 5BCCAE60
-P 7400 4300
-AR Path="/5BC99DB9/5BCCAE60" Ref="SJ?"  Part="1"
-AR Path="/5BCA1914/5BCCAE60" Ref="SJ15"  Part="1"
-F 0 "SJ15" H 7300 4400 59  0000 L BNN
-F 1 "SOLDERJUMPER" H 7300 4150 59  0000 L BNN
-F 2 "Adafruit MAX31865:SOLDERJUMPER_ARROW_NOPASTE" H 7400 4300 50  0001 C CNN
-F 3 "" H 7400 4300 50  0001 C CNN
-	1    7400 4300
-	0    -1   -1   0
-$EndComp
-$Comp
-L Connector_Generic:Conn_01x04 J?
-U 1 1 5BCCAE67
-P 8100 3400
-AR Path="/5BC99DB9/5BCCAE67" Ref="J?"  Part="1"
-AR Path="/5BCA1914/5BCCAE67" Ref="J6"  Part="1"
-F 0 "J6" H 8180 3392 50  0000 L CNN
-F 1 "Conn_01x04" H 8180 3301 50  0000 L CNN
-F 2 "TerminalBlock_4Ucon:TerminalBlock_4Ucon_1x04_P3.50mm_Horizontal" H 8100 3400 50  0001 C CNN
-F 3 "~" H 8100 3400 50  0001 C CNN
-	1    8100 3400
-	1    0    0    -1
-$EndComp
-Wire Wire Line
-	7700 4100 7700 3500
-Wire Wire Line
-	7600 4200 7800 4200
-Wire Wire Line
-	7800 4200 7800 3600
-Wire Wire Line
-	7800 3600 7900 3600
-Wire Wire Line
-	7700 3500 7900 3500
-Wire Wire Line
-	7600 3400 7900 3400
-Wire Wire Line
-	7400 3300 7900 3300
+	6200 2500 6400 2500
+Wire Wire Line
+	6400 2500 6900 2500
+Wire Wire Line
+	6200 2700 6400 2700
+Wire Wire Line
+	6400 2700 6400 2500
+Connection ~ 6400 2500
+Wire Wire Line
+	6200 2900 6900 2900
+Wire Wire Line
+	6200 3100 6900 3100
+Wire Wire Line
+	6900 3100 6900 2900
+Connection ~ 6900 2900
+Wire Wire Line
+	6200 3700 6400 3700
+Wire Wire Line
+	6400 3800 6400 3700
+Wire Wire Line
+	7000 4200 6400 4200
+Wire Wire Line
+	6400 4100 6400 4200
+Connection ~ 6400 4200
+$Comp
+L Adafruit_MAX31865-eagle-import:RESISTOR0805_NOOUTLINE R?
+U 1 1 5E67B9ED
+P 6900 2700
+AR Path="/5BC99DB9/5E67B9ED" Ref="R?"  Part="1"
+AR Path="/5BCA1911/5E67B9ED" Ref="R?"  Part="1"
+AR Path="/5BCA1914/5E67B9ED" Ref="R20"  Part="1"
+F 0 "R20" H 6900 2800 50  0000 C CNN
+F 1 "430Ω / 4300Ω 0.1%" H 6900 2600 40  0000 C CNB
+F 2 "Adafruit MAX31865:0805-NO" H 6900 2700 50  0001 C CNN
+F 3 "" H 6900 2700 50  0001 C CNN
+	1    6900 2700
+	0    -1   -1   0
+$EndComp
+$Comp
+L Adafruit_MAX31865-eagle-import:CAP_CERAMIC0805-NOOUTLINE C?
+U 1 1 5E67B9F3
+P 6400 4000
+AR Path="/5BC99DB9/5E67B9F3" Ref="C?"  Part="1"
+AR Path="/5BCA1911/5E67B9F3" Ref="C?"  Part="1"
+AR Path="/5BCA1914/5E67B9F3" Ref="C17"  Part="1"
+F 0 "C17" V 6310 4049 50  0000 C CNN
+F 1 "100nF" V 6490 4049 50  0000 C CNN
+F 2 "Adafruit MAX31865:0805-NO" H 6400 4000 50  0001 C CNN
+F 3 "" H 6400 4000 50  0001 C CNN
+	1    6400 4000
+	1    0    0    -1
+$EndComp
+Text Notes 7100 2800 0    59   ~ 0
+R1 = 4x RTD resistance at 0°C (so 400 ohm for a 100 ohm RTD).\nUse high quality 1% or better resistors
+Wire Wire Line
+	6200 4200 6400 4200
+Wire Wire Line
+	6400 3700 7000 3700
+Connection ~ 6400 3700
+Wire Wire Line
+	6200 3300 7000 3300
+Wire Wire Line
+	6200 4400 7000 4400
+Text GLabel 7000 3300 2    50   Input ~ 0
+O33
+Text GLabel 7000 3700 2    50   Input ~ 0
+O35
+Text GLabel 7000 4200 2    50   Input ~ 0
+O37
+Text GLabel 7000 4400 2    50   Input ~ 0
+O39
+NoConn ~ 6200 3500
 $EndSCHEMATC
