File: PCB/mosfet_switch.sch (KiCad schematic (older format))
At the start: 4 parts, among them Q1 DMN1150UFB-7B, Q2 NVTR0202PLT1G

Commit message: Patrick: fixed wrong ground/source assignment of mosfet switch.
Connections:
- net GPIO_3V3: now also Q1.2 (S), R46.1; no longer Q1.1 (G), R46.2
- new net: Q1.1 (G), R46.2
Changed lines of the file:
@@
 	1    0    0    -1
 $EndComp
-Text GLabel 5000 4000 0    50   Input ~ 0
+Text GLabel 6000 4600 3    50   Input ~ 0
 GPIO_3V3
 $Comp
@@
 L Adafruit_MAX31865-eagle-import:GND #0111
 U 1 1 5E62A8A8
-P 6000 4700
-F 0 "#0111" H 6050 4750 50  0001 C CNN
-F 1 "GND" H 6078 4738 42  0000 L CNN
-F 2 "" H 6000 4700 50  0001 C CNN
-F 3 "" H 6000 4700 50  0001 C CNN
-	1    6000 4700
-	1    0    0    -1
+P 4900 4000
+F 0 "#0111" H 4950 4050 50  0001 C CNN
+F 1 "GND" H 4978 4038 42  0000 L CNN
+F 2 "" H 4900 4000 50  0001 C CNN
+F 3 "" H 4900 4000 50  0001 C CNN
+	1    4900 4000
+	0    1    1    0
 $EndComp
 Wire Wire Line
-	5400 4000 5000 4000
-Connection ~ 5400 4000
+	5000 4000 5400 4000
 $Comp
 L FDN360P:NVTR0202PLT1G Q2
@@
 	6000 4400 6000 4500
 Connection ~ 6000 4500
+Connection ~ 5400 4000
 $EndSCHEMATC
